File: pcb/DisplayAdapter_DOGM128.kicad_pcb (KiCad board)
At the start: 2 copper layers, 69.3 x 47.4 mm, 26 parts, among them J1 Connector, Q1 IRLML2502, U2 BCR42XUW6, U3 BCR42XUW6, U4 BCR42XUW6

Commit message: Revision 2
Parts:
- removed J1: Connector, Connector_PinHeader_2.54mm:PinHeader_1x08_P2.54mm_Vertical
- removed R1, R2: 90Ω, Resistor_SMD:R_0805_2012Metric_Pad1.20x1.40mm_HandSolder
- removed U2, U3: BCR42XUW6, Package_TO_SOT_SMD:SOT-23-6
- added J101: Conn_01x09_Male, Connector_PinHeader_2.54mm:PinHeader_1x09_P2.54mm_Horizontal, B.Cu at (95.9, 47.9)
- R3: value 90Ω -> 80Ω
- moved Q1 13.7 mm to (143.8, 73.4)
Connections:
- U4 pad 2: Net-(U1-Pad20) -> Net-(U1-Pad18)
- U4 pad 3: Net-(U1-Pad20) -> Net-(U1-Pad18)
- U4 pad 5: Net-(U1-Pad20) -> Net-(U1-Pad18)
- U? pad 1: /3V3 -> Net-(U1-Pad1)
- U? pad 19: Net-(U1-Pad19) -> Net-(U1-Pad18)
- U? pad 2: /3V3 -> Net-(U1-Pad1)
- U? pad 20: Net-(U1-Pad20) -> Net-(U1-Pad18)
- U? pad 3: /3V3 -> Net-(U1-Pad1)
Routing:
- net Net-(Q1-Pad2): track 19.1 -> 3.45 mm
- net Net-(U1-Pad19): track 12.9 -> 0.00 mm
- net /DISP_BKLT: track 40.8 -> 52.5 mm
- net Net-(U1-Pad20): track 10.6 -> 0.00 mm
- net Net-(U1-Pad1): track 0.00 -> 5.08 mm
- net Net-(U1-Pad18): track 17.4 -> 14.8 mm
- net Net-(R2-Pad1): track 2.19 -> 0.00 mm
- net Net-(R1-Pad1): track 2.19 -> 0.00 mm
Other:
- board text added: "3V3 5V ~{CS1B} ~{RESET} A0 SCK MOSI DISP_BKLT GND"
- board text added: "Display Adapter EA_DOGM128 Rev 2"
- board text removed: "3V3 DISP_ES DISP_RESET A0 SCK MOSI DISP_BKLT GND"
- board text removed: "Display Adapter EA_DOGM128 Rev 1"
