File: pcb/DisplayAdapter_DOGM128.kicad_sch (KiCad schematic)
At the start: 26 parts, among them J1 Connector, Q1 IRLML2502, U1 EA_DOGM128X-6, U2 BCR42XUW6, U3 BCR42XUW6, U4 BCR42XUW6

Commit message: Revision 2
Parts:
- removed J1: Connector, Connector_PinHeader_2.54mm:PinHeader_1x08_P2.54mm_Vertical, symbol Connector:Conn_01x08_Male
- removed R1, R2: 90Ω, Resistor_SMD:R_0805_2012Metric_Pad1.20x1.40mm_HandSolder, symbol Device:R
- removed U2, U3: BCR42XUW6, Package_TO_SOT_SMD:SOT-23-6, symbol DisplayAdapter_DOGM128:BCR42XUW6
- added J101: Conn_01x09_Male, Connector_PinHeader_2.54mm:PinHeader_1x09_P2.54mm_Horizontal, symbol Connector:Conn_01x09_Male
- R3: value 90Ω -> 80Ω
Connections:
- net 3V3: now also J101.1 (Pin_1); no longer U1.1 (A1+), U1.2 (A2+), U1.3 (A3+)
- net A0: now also J101.5 (Pin_5)
- net DISP_BKLT: now also J101.8 (Pin_8)
- net GND: now also J101.9 (Pin_9)
- net MOSI: now also J101.7 (Pin_7)
- net SCK: now also J101.6 (Pin_6)
- net ~{DISP_CS}: now also J101.3 (Pin_3)
- net ~{DISP_REST}: now also J101.4 (Pin_4)
- net at U1.18 (C1-): now also U1.19 (C2-), U1.20 (C3-), U4.2 (OUT), U4.3 (OUT), U4.5 (OUT)
- new net: U1.1 (A1+), U1.2 (A2+), U1.3 (A3+)
- new net 5V: J101.2 (Pin_2)
Other:
- note added: "1.4 V_{OUT}"
- note added: "Backlight V_{f} = 3.3V"
- note added: "R_{EXT} Limit to 20mA"
- moved on the sheet: R3, U4
